Commit message: update urdf

File: humanoid_description/urdf/humanoid.urdf (robot description, URDF)
Before this commit: robot humanoid, 12 links, 11 joints
Links:
- link base_link: mass 1.41235892615924 -> 1.36479420298455
- link left_hip_pitch_link: mass 0.181404797807314 -> 0.184010633558111
- link left_hip_roll_link: mass 0.313038507460088 -> 0.314265384083357
- link left_knee_link: mass 0.1298788192464 -> 0.129468515543408
- link right_hip_pitch_link: mass 0.176757480845002 -> 0.177043458080398
- link right_hip_roll_link: mass 0.313038507460088 -> 0.314265384083356
- link right_hip_yaw_link: mass 0.0261773071845988 -> 0.141006445664123
- link right_knee_link: mass 0.129878818884871 -> 0.12946851518188
Joints:
- joint left_ankle_joint: axis 0.251595646506534 0 0.967832439350407 -> 0 0 1; origin xyz=0.15 -0.00910507425656893 0 rpy=0 0 -1.5707963267949 -> xyz=0.15 -0.0091051 0 rpy=0 0 -1.5708
- joint left_hip_pitch_joint: origin xyz=0 0.011726065302402 0.0440174865902528 rpy=1.5707963267949 0 0 -> xyz=0 0.013726 0.044017 rpy=1.5708 0 0
- joint left_hip_roll_joint: axis 0 0 -1 -> 0 0 1; origin xyz=-0.0145174865902528 -0.003773934697598 0.0518623737059448 rpy=0 -1.5707963267949 0 -> xyz=-0.014517 -0.0037739 0.051862 rpy=3.14 -1.5708 0
- joint left_hip_yaw_joint: axis 0 0 -1 -> 0 0 1; origin xyz=-0.0875 0 0 rpy=3.14159265358979 0 1.5707963267949 -> xyz=-0.0875 0 0 rpy=3.1416 0 1.5708
- joint left_knee_joint: origin xyz=0.149999999999999 0 0.0144999999999998 rpy=-3.14159265358979 0 0 -> xyz=0.15 0 0.0165 rpy=-3.1416 0 0
- joint right_ankle_joint: origin xyz=0.15 0 0 rpy=0 0 -1.5707963267949 -> xyz=0.15 0 0 rpy=0 0 -1.5708
- joint right_hip_pitch_joint: origin xyz=0 0.0155000000000001 0.0445 rpy=1.5707963267949 0 0 -> xyz=0 0.0175 0.0445 rpy=1.5708 0 0
- joint right_hip_roll_joint: axis 0 0 -1 -> 0 0 1; origin xyz=-0.015 0 0.0518623737059446 rpy=0 -1.5707963267949 0 -> xyz=-0.015 0 0.051862 rpy=3.14 -1.5708 0
- joint right_hip_yaw_joint: axis 0 0 -1 -> 0 0 1; origin xyz=0.0875 0 0 rpy=3.14159265358979 0 1.5707963267949 -> xyz=0.0875 0 0 rpy=3.1416 0 1.5708
- joint right_knee_joint: axis 0 0 -1 -> 0 0 1; origin xyz=0.15 0 0.0145000000000002 rpy=3.14159265358979 0 0 -> xyz=0.15 0 0.0165 rpy=3.1416 0 0
